File: Hardware/Chipshouter-cat.kicad_sch (KiCad schematic)
At the start: 72 parts

Commit message: All schematic added
Parts:
- removed D6: (no value), symbol Diode:MBR340
- removed R12: (no value), symbol Device:R_Small
- added D?: (no value), symbol Diode:MBR340
- C10, C11, C12, C14, C15, C16, C17, C18, C19, C20, C7, C8, U2, Y1: Stock en EC No -> (none)
- C13, C9, R17, R18, R19, R20: Stock en EC Yes -> (none)
- U3: Manf# (none) -> RPI Chip RP2040-7-500; Proveedor (none) -> MOUSER; Stock en EC Yes -> (none)
Connections:
- net A2 is gone; now on net GP28: U3.40 (GPIO28_ADC2)
- net D0 is gone; now on net GP5: U3.7 (GPIO5)
- net D10 is gone; now on net GP11: U3.14 (GPIO11)
- net D12 is gone; now on net GP20: U3.31 (GPIO20)
- net GPIO18 is gone; now on net CHARGED: U3.29 (GPIO18)
- net RX is gone; now on net GP1: U3.3 (GPIO1)
- net SCL is gone; now on net GP3: U3.5 (GPIO3)
- net SDA is gone; now on net GP2: U3.4 (GPIO2)
- net TX is gone; now on net GP0: U3.2 (GPIO0)
- net +3V3: now also D?.2 (A)
- net CHARGED: now also U3.38 (GPIO26_ADC0)
- net GP14: now also U3.17 (GPIO14)
- net GP27: now also U3.39 (GPIO27_ADC1)
- net GP4: now also U3.6 (GPIO4)
- net GP6: now also U3.8 (GPIO6)
- net GP7: now also U3.9 (GPIO7)
- net VBUS: now also SW2.1 (A)
- net VSYS: now also D?.1 (K)
- net CLK: no longer names the net of U3.35 (GPIO23)
- net D11: no longer names the net of U3.15 (GPIO12)
- net D13: no longer names the net of U3.32 (GPIO21)
- net D24: no longer names the net of U3.36 (GPIO24)
- net D25: no longer names the net of U3.37 (GPIO25)
- net D5: no longer names the net of U3.11 (GPIO8)
- net D6: no longer names the net of U3.12 (GPIO9)
- net D9: no longer names the net of U3.13 (GPIO10)
- net DOUT: no longer names the net of U3.34 (GPIO22)
- net GPIO13: no longer names the net of U3.16 (GPIO13)
- net GPIO17: no longer names the net of U3.28 (GPIO17)
- no-connect marks 12 -> 2
Other:
- moved on the sheet: C10, C5, C6, C8, R18, R19, R20, SW2, U1, U3, Y1

Commit message: BOM and footprints added
Parts:
- added F1: (no value), symbol Device:Fuse_Small
- C10, C8: Manf# (none) -> C0603C270J5GAC7411; Proveedor (none) -> MOUSER
- C11, C12, C14, C15, C16, C17, C18, C19, C20, C7: Manf# (none) -> CC0402ZRY5V7BB104; Proveedor (none) -> MOUSER
- C13, C9: LCSC# C696901 -> (none); Manf# (none) -> CL10A105KP8NNNC; Proveedor (none) -> MOUSER
- C5, C6: LCSC# C85713 -> (none); Manf# (none) -> CL05A106MQ5NUNC; Proveedor (none) -> MOUSER
- D6: renamed from D?; LCSC# C130880 -> C81143; Proveedor (none) -> LCSC
- J1: LCSC# C530661 -> (none)
- R17: LCSC# (none) -> C99198; Proveedor (none) -> LCSC
- R18: LCSC# (none) -> C115325; Proveedor (none) -> LCSC
- R19, R20: Manf# (none) -> ERJ-3GEYJ270V; Proveedor (none) -> MOUSER
- SW2: Manf# (none) -> JS102011SAQN; Proveedor (none) -> MOUSER
- SW4, SW5: LCSC# C2886897 -> (none); Manf# (none) -> TL3342F450QG; Proveedor (none) -> MOUSER
- U1: LCSC# - -> (none); Manf# (none) -> AP7347DQ-33W5-7; Proveedor (none) -> MOUSER
- U2: Manf# (none) -> W25Q16JVUUIQ TR; Proveedor (none) -> MOUSER
- Y1: LCSC# (none) -> C709001; Proveedor (none) -> LCSC
Connections:
- net DM is gone; now on net D-: P1.A7 (D-)
- net DP is gone; now on net D+: P1.A6 (D+)
- net VSYS is gone; now on net +3V3: D10.1 (K), D6.1 (K)
- net +3V3: no longer C6.1, D6.2 (A), U1.5 (VOUT)
- net VBUS: now also F1.2; no longer P1.A4 (VBUS), P1.A9 (VBUS), P1.B4 (VBUS), P1.B9 (VBUS)
- net RD+: no longer names the net of R19.2, U3.47 (USB_DP)
- net RD-: no longer names the net of R20.2, U3.46 (USB_DM)
- new net: F1.1, P1.A4 (VBUS), P1.A9 (VBUS), P1.B4 (VBUS), P1.B9 (VBUS)
- new net: C6.1, D6.2 (A), U1.5 (VOUT)
Other:
- moved on the sheet: C5, C6, D6, SW2, U1
