File: Hardware/BuggyCat.kicad_sch (KiCad schematic)
At the start: 74 parts, among them J1 Antenna, J2 BG306-02-A-2-0400-L-G, J3 Header7, J4 Header 2, J5 Header 4, J6 Input Power:2x AA Battery, P1 USB_C_Plug_USB2.0, Q1 AO3422, Q1 DMG3415U-7, Q2 AO3422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

Commit message: Reassigned footprints and 3d models
Parts:
- C4: footprint chipshouter:CAPC6153X500N -> BuggyCat:CAPC6153X500N
- J1: footprint chipshouter:732511150 -> BuggyCat:732511150
- J2: footprint chipshouter:BG30602A20400LG -> BuggyCat:BG30602A20400LG
- J6: footprint chipshouter:JST_S2B-PH-K-S(LF)(SN) -> BuggyCat:JST_S2B-PH-K-S(LF)(SN)
- Q3: footprint chipshouter:SOP254P952X470-6N -> BuggyCat:SOP254P952X470-6N
- R11: footprint chipshouter:RESC6432X120N -> BuggyCat:RESC6432X120N
- T1, T2: footprint chipshouter:ATB3225240110T000 -> BuggyCat:ATB3225240110T000
- U2: footprint chipshouter:W25Q16JVUUIQ -> BuggyCat:W25Q16JVUUIQ
- U3: footprint chipshouter:RP2040-QFN-56 -> BuggyCat:RP2040-QFN-56
