File: Hardware/BuggyCat.kicad_sch (KiCad schematic)
At the start: 74 parts, among them J1 Antenna, J2 BG306-02-A-2-0400-L-G, J3 Header7, J4 Header 2, J5 Header 4, J6 Input Power:2x AA Battery, P1 USB_C_Plug_USB2.0, Q1 AO3422, Q1 DMG3415U-7, Q2 AO3422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

Commit message: Add to BOM components of LCSC
Parts:
- C1, C3: LCSC# (none) -> C98192
- C10, C8: LCSC# (none) -> C107045
- C11, C12, C14, C15, C16, C17, C18, C19, C20, C7: LCSC# (none) -> C106209
- C13, C9: LCSC# (none) -> C26413
- C2: LCSC# (none) -> C30926
- C5, C6: LCSC# (none) -> C15525
- D4: LCSC# (none) -> C85095
- D7, D9: LCSC# (none) -> C157740
- D8: LCSC# (none) -> C192666
- F1: LCSC# - -> C2649565
- Q1, Q2: LCSC# (none) -> C37130
- R1, R9: LCSC# (none) -> C109318
- R13, R14, R16, R5, R6: LCSC# (none) -> C22548
- R19, R20: LCSC# (none) -> C25224
- R2, R4: LCSC# (none) -> C23186
- R3: LCSC# (none) -> C141697
- R7: LCSC# (none) -> C114065
- R8: LCSC# (none) -> C114572
- SW1, SW3, SW4, SW5, SW6: LCSC# (none) -> C2886897
- SW2: LCSC# - -> C221829
- T1, T2: LCSC# (none) -> C249001
- U1: LCSC# (none) -> C216640
Changed lines of the file:
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@@
       (effects (font (size 1.27 1.27)) hide)
     )
-    (property "LCSC#" "" (at 353.695 235.331 0)
+    (property "LCSC#" "C106209" (at 353.695 235.331 0)
       (effects (font (size 1.27 1.27)) hide)
     )
@@
       (effects (font (size 1.27 1.27)) hide)
     )
+    (property "LCSC#" "C109318" (at 41.275 136.525 0)
+      (effects (font (size 1.27 1.27)) hide)
+    )
     (pin "1")
     (pin "2")
@@
       (effects (font (size 1.27 1.27)) hide)
     )
+    (property "LCSC#" "C23186" (at 45.085 244.475 0)
+      (effects (font (size 1.27 1.27)) hide)
+    )
     (pin "1")
     (pin "2")
@@
       (effects (font (size 1.27 1.27)) hide)
     )
-    (property "LCSC#" "" (at 164.973 272.542 0)
+    (property "LCSC#" "C15525" (at 164.973 272.542 0)
       (effects (font (size 1.27 1.27)) hide)
     )
@@
       (effects (font (size 1.27 1.27)) hide)
     )
+    (property "LCSC#" "C2886897" (at 125.73 31.75 0)
+      (effects (font (size 1.27 1.27)) hide)
+    )
     (pin "1")
     (pin "2")
@@
       (effects (font (size 1.27 1.27)) hide)
     )
-    (property "LCSC#" "" (at 211.455 276.987 0)
+    (property "LCSC#" "C2886897" (at 211.455 276.987 0)
       (effects (font (size 1.27 1.27)) hide)
     )
@@
       (effects (font (size 1.27 1.27)) hide)
     )
+    (property "LCSC#" "C23186" (at 50.8 247.015 0)
+      (effects (font (size 1.27 1.27)) hide)
+    )
     (pin "1")
     (pin "2")
@@
       (effects (font (size 1.27 1.27)) hide)
     )
+    (property "LCSC#" "C30926" (at 75.565 154.305 0)
+      (effects (font (size 1.27 1.27)) hide)
+    )
     (pin "1")
     (pin "2")
@@
       (effects (font (size 1.27 1.27)) hide)
     )
-    (property "LCSC#" "" (at 398.78 120.65 0)
+    (property "LCSC#" "C25224" (at 398.78 120.65 0)
       (effects (font (size 1.27 1.27)) hide)
     )
@@
       (effects (font (size 1.27 1.27)) hide)
     )
+    (property "LCSC#" "C114572" (at 108.585 127 0)
+      (effects (font (size 1.27 1.27)) hide)
+    )
     (pin "1")
     (pin "2")
@@
       (effects (font (size 1.27 1.27)) hide)
     )
+    (property "LCSC#" "C157740" (at 199.39 63.5 0)
+      (effects (font (size 1.27 1.27)) hide)
+    )
     (pin "1")
     (pin "2")
@@
       (effects (font (size 1.27 1.27)) hide)
     )
-    (property "LCSC#" "-" (at 44.45 239.395 0)
+    (property "LCSC#" "C2649565" (at 44.45 239.395 0)
       (effects (font (size 1.27 1.27)) hide)
     )
@@
       (effects (font (size 1.27 1.27)) hide)
     )
+    (property "LCSC#" "C37130" (at 63.5 100.965 0)
+      (effects (font (size 1.27 1.27)) hide)
+    )
     (pin "1")
     (pin "2")
@@
       (effects (font (size 1.27 1.27)) hide)
     )
-    (property "LCSC#" "" (at 313.309 235.077 0)
+    (property "LCSC#" "C26413" (at 313.309 235.077 0)
       (effects (font (size 1.27 1.27)) hide)
     )
@@
       (effects (font (size 1.27 1.27)) hide)
     )
+    (property "LCSC#" "C22548" (at 210.185 71.12 0)
+      (effects (font (size 1.27 1.27)) hide)
+    )
     (pin "1")
     (pin "2")
@@
       (effects (font (size 1.27 1.27)) hide)
     )
+    (property "LCSC#" "C22548" (at 52.07 154.305 0)
+      (effects (font (size 1.27 1.27)) hide)
+    )
     (pin "1")
     (pin "2")
@@
       (effects (font (size 1.27 1.27)) hide)
     )
+    (property "LCSC#" "C192666" (at 199.39 71.12 0)
+      (effects (font (size 1.27 1.27)) hide)
+    )
     (pin "1")
     (pin "2")
@@
       (effects (font (size 1.27 1.27)) hide)
     )
-    (property "LCSC#" "" (at 346.075 235.331 0)
+    (property "LCSC#" "C26413" (at 346.075 235.331 0)
       (effects (font (size 1.27 1.27)) hide)
     )
@@
       (effects (font (size 1.27 1.27)) hide)
     )
-    (property "LCSC#" "" (at 321.437 235.077 0)
+    (property "LCSC#" "C106209" (at 321.437 235.077 0)
       (effects (font (size 1.27 1.27)) hide)
     )
@@
       (effects (font (size 1.27 1.27)) hide)
     )
-    (property "LCSC#" "" (at 299.085 178.054 0)
+    (property "LCSC#" "C107045" (at 299.085 178.054 0)
       (effects (font (size 1.27 1.27)) hide)
     )
@@
       (effects (font (size 1.27 1.27)) hide)
     )
+    (property "LCSC#" "C249001" (at 94.742 76.327 0)
+      (effects (font (size 1.27 1.27)) hide)
+    )
     (pin "1")
     (pin "2")
@@
       (effects (font (size 1.27 1.27)) hide)
     )
-    (property "LCSC#" "" (at 391.795 235.331 0)
+    (property "LCSC#" "C106209" (at 391.795 235.331 0)
       (effects (font (size 1.27 1.27)) hide)
     )
@@
       (effects (font (size 1.27 1.27)) hide)
     )
-    (property "LCSC#" "" (at 361.061 235.331 0)
+    (property "LCSC#" "C106209" (at 361.061 235.331 0)
       (effects (font (size 1.27 1.27)) hide)
     )
@@
       (effects (font (size 1.27 1.27)) hide)
     )
-    (property "LCSC#" "" (at 399.415 235.077 0)
+    (property "LCSC#" "C106209" (at 399.415 235.077 0)
       (effects (font (size 1.27 1.27)) hide)
     )
@@
       (effects (font (size 1.27 1.27)) hide)
     )
-    (property "LCSC#" "" (at 368.681 235.331 0)
+    (property "LCSC#" "C106209" (at 368.681 235.331 0)
       (effects (font (size 1.27 1.27)) hide)
     )
@@
       (effects (font (size 1.27 1.27)) hide)
     )
-    (property "LCSC#" "" (at 311.785 178.689 0)
+    (property "LCSC#" "C107045" (at 311.785 178.689 0)
       (effects (font (size 1.27 1.27)) hide)
     )
@@
       (effects (font (size 1.27 1.27)) hide)
     )
-    (property "LCSC#" "" (at 398.78 118.11 0)
+    (property "LCSC#" "C25224" (at 398.78 118.11 0)
       (effects (font (size 1.27 1.27)) hide)
     )
@@
       (effects (font (size 1.27 1.27)) hide)
     )
+    (property "LCSC#" "C2886897" (at 255.27 28.575 0)
+      (effects (font (size 1.27 1.27)) hide)
+    )
     (pin "1")
     (pin "2")
@@
       (effects (font (size 1.27 1.27)) hide)
     )
+    (property "LCSC#" "C85095" (at 110.744 66.675 0)
+      (effects (font (size 1.27 1.27)) hide)
+    )
     (pin "1")
     (pin "2")
@@
       (effects (font (size 1.27 1.27)) hide)
     )
-    (property "LCSC#" "" (at 328.549 235.077 0)
+    (property "LCSC#" "C106209" (at 328.549 235.077 0)
       (effects (font (size 1.27 1.27)) hide)
     )
@@
       (effects (font (size 1.27 1.27)) hide)
     )
-    (property "LCSC#" "" (at 384.175 235.331 0)
+    (property "LCSC#" "C106209" (at 384.175 235.331 0)
       (effects (font (size 1.27 1.27)) hide)
     )
@@
       (effects (font (size 1.27 1.27)) hide)
     )
-    (property "LCSC#" "-" (at 156.21 267.97 0)
+    (property "LCSC#" "C221829" (at 156.21 267.97 0)
       (effects (font (size 1.27 1.27)) hide)
     )
@@
       (effects (font (size 1.27 1.27)) hide)
     )
-    (property "LCSC#" "" (at 210.82 264.922 0)
+    (property "LCSC#" "C2886897" (at 210.82 264.922 0)
       (effects (font (size 1.27 1.27)) hide)
     )
@@
       (effects (font (size 1.27 1.27)) hide)
     )
+    (property "LCSC#" "C114065" (at 66.675 40.64 0)
+      (effects (font (size 1.27 1.27)) hide)
+    )
     (pin "1")
     (pin "2")
@@
       (effects (font (size 1.27 1.27)) hide)
     )
-    (property "LCSC#" "" (at 376.301 235.331 0)
+    (property "LCSC#" "C106209" (at 376.301 235.331 0)
       (effects (font (size 1.27 1.27)) hide)
     )
@@
       (effects (font (size 1.27 1.27)) hide)
     )
-    (property "LCSC#" "" (at 235.585 273.177 0)
+    (property "LCSC#" "C106209" (at 235.585 273.177 0)
       (effects (font (size 1.27 1.27)) hide)
     )
@@
       (effects (font (size 1.27 1.27)) hide)
     )
+    (property "LCSC#" "C109318" (at 117.475 120.65 0)
+      (effects (font (size 1.27 1.27)) hide)
+    )
     (pin "1")
     (pin "2")
@@
       (effects (font (size 1.27 1.27)) hide)
     )
-    (property "LCSC#" "" (at 189.865 272.415 0)
+    (property "LCSC#" "C15525" (at 189.865 272.415 0)
       (effects (font (size 1.27 1.27)) hide)
     )
@@
       (effects (font (size 1.27 1.27)) hide)
     )
+    (property "LCSC#" "C22548" (at 210.185 63.5 0)
+      (effects (font (size 1.27 1.27)) hide)
+    )
     (pin "1")
     (pin "2")
@@
       (effects (font (size 1.27 1.27)) hide)
     )
-    (property "LCSC#" "" (at 179.705 270.51 0)
+    (property "LCSC#" "C216640" (at 179.705 270.51 0)
       (effects (font (size 1.27 1.27)) hide)
     )
@@
       (effects (font (size 1.27 1.27)) hide)
     )
+    (property "LCSC#" "C2886897" (at 203.2 85.09 0)
+      (effects (font (size 1.27 1.27)) hide)
+    )
     (pin "1")
     (pin "2")
@@
       (effects (font (size 1.27 1.27)) hide)
     )
+    (property "LCSC#" "C98192" (at 82.677 98.425 0)
+      (effects (font (size 1.27 1.27)) hide)
+    )
     (pin "1")
     (pin "2")
@@
       (effects (font (size 1.27 1.27)) hide)
     )
+    (property "LCSC#" "C141697" (at 49.53 86.995 0)
+      (effects (font (size 1.27 1.27)) hide)
+    )
     (pin "1")
     (pin "2")
@@
       (effects (font (size 1.27 1.27)) hide)
     )
+    (property "LCSC#" "C37130" (at 63.5 147.955 0)
+      (effects (font (size 1.27 1.27)) hide)
+    )
     (pin "1")
     (pin "2")
@@
       (effects (font (size 1.27 1.27)) hide)
     )
+    (property "LCSC#" "C98192" (at 73.152 98.425 0)
+      (effects (font (size 1.27 1.27)) hide)
+    )
     (pin "1")
     (pin "2")
@@
       (effects (font (size 1.27 1.27)) hide)
     )
+    (property "LCSC#" "C22548" (at 52.705 106.045 0)
+      (effects (font (size 1.27 1.27)) hide)
+    )
     (pin "1")
     (pin "2")
@@
       (effects (font (size 1.27 1.27)) hide)
     )
+    (property "LCSC#" "C249001" (at 82.55 125.73 0)
+      (effects (font (size 1.27 1.27)) hide)
+    )
     (pin "1")
     (pin "2")
@@
       (effects (font (size 1.27 1.27)) hide)
     )
+    (property "LCSC#" "C157740" (at 255.905 41.275 0)
+      (effects (font (size 1.27 1.27)) hide)
+    )
     (pin "1")
     (pin "2")
@@
       (effects (font (size 1.27 1.27)) hide)
     )
+    (property "LCSC#" "C22548" (at 244.475 41.275 0)
+      (effects (font (size 1.27 1.27)) hide)
+    )

Commit message: SW1, SW3 and SW6 buttons changed
Parts:
- SW1, SW3, SW6: value TL3342F450QG -> TL3305AF260QG; footprint Button_Switch_SMD:SW_SPST_TL3342 -> BuggyCat:TL3305AF160QG; LCSC# C2886897 -> (none); Manf# TL3342F450QG -> TL3305AF260QG
Changed lines of the file:
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@@
       (effects (font (size 1.27 1.27)))
     )
-    (property "Value" "TL3342F450QG" (at 125.73 26.67 0)
-      (effects (font (size 1.27 1.27)))
-    )
-    (property "Footprint" "Button_Switch_SMD:SW_SPST_TL3342" (at 125.73 26.67 0)
-      (effects (font (size 1.27 1.27)) hide)
-    )
-    (property "Datasheet" "https://www.mouser.mx/datasheet/2/140/ESwitch_2623_TL3301-3103205.pdf" (at 125.73 26.67 0)
-      (effects (font (size 1.27 1.27)) hide)
-    )
-    (property "Manf#" "TL3342F450QG" (at 125.73 31.75 0)
+    (property "Value" "TL3305AF260QG" (at 125.73 26.67 0)
+      (effects (font (size 1.27 1.27)))
+    )
+    (property "Footprint" "BuggyCat:TL3305AF160QG" (at 125.73 26.67 0)
+      (effects (font (size 1.27 1.27)) hide)
+    )
+    (property "Datasheet" "https://www.mouser.mx/datasheet/2/140/TL3305-2065758.pdf" (at 125.73 26.67 0)
+      (effects (font (size 1.27 1.27)) hide)
+    )
+    (property "Manf#" "TL3305AF260QG" (at 125.73 31.75 0)
       (effects (font (size 1.27 1.27)) hide)
     )
@@
       (effects (font (size 1.27 1.27)) hide)
     )
-    (property "LCSC#" "C2886897" (at 125.73 31.75 0)
+    (property "LCSC#" "" (at 125.73 31.75 0)
       (effects (font (size 1.27 1.27)) hide)
     )
@@
       (effects (font (size 1.27 1.27)))
     )
-    (property "Value" "TL3342F450QG" (at 255.27 23.495 0)
-      (effects (font (size 1.27 1.27)))
-    )
-    (property "Footprint" "Button_Switch_SMD:SW_SPST_TL3342" (at 255.27 23.495 0)
-      (effects (font (size 1.27 1.27)) hide)
-    )
-    (property "Datasheet" "https://www.mouser.mx/datasheet/2/240/ksc7-3050369.pdf" (at 255.27 23.495 0)
-      (effects (font (size 1.27 1.27)) hide)
-    )
-    (property "Manf#" "TL3342F450QG" (at 255.27 28.575 0)
+    (property "Value" "TL3305AF260QG" (at 255.27 23.495 0)
+      (effects (font (size 1.27 1.27)))
+    )
+    (property "Footprint" "BuggyCat:TL3305AF160QG" (at 255.27 23.495 0)
+      (effects (font (size 1.27 1.27)) hide)
+    )
+    (property "Datasheet" "https://www.mouser.mx/datasheet/2/140/TL3305-2065758.pdf" (at 255.27 23.495 0)
+      (effects (font (size 1.27 1.27)) hide)
+    )
+    (property "Manf#" "TL3305AF260QG" (at 255.27 28.575 0)
       (effects (font (size 1.27 1.27)) hide)
     )
@@
       (effects (font (size 1.27 1.27)) hide)
     )
-    (property "LCSC#" "C2886897" (at 255.27 28.575 0)
+    (property "LCSC#" "" (at 255.27 28.575 0)
       (effects (font (size 1.27 1.27)) hide)
     )
@@
       (effects (font (size 1.27 1.27)))
     )
-    (property "Value" "TL3342F450QG" (at 203.2 80.01 0)
-      (effects (font (size 1.27 1.27)))
-    )
-    (property "Footprint" "Button_Switch_SMD:SW_SPST_TL3342" (at 203.2 80.01 0)
-      (effects (font (size 1.27 1.27)) hide)
-    )
-    (property "Datasheet" "https://www.mouser.mx/datasheet/2/240/ksc7-3050369.pdf" (at 203.2 80.01 0)
-      (effects (font (size 1.27 1.27)) hide)
-    )
-    (property "Manf#" "TL3342F450QG" (at 203.2 85.09 0)
+    (property "Value" "TL3305AF260QG" (at 203.2 80.01 0)
+      (effects (font (size 1.27 1.27)))
+    )
+    (property "Footprint" "BuggyCat:TL3305AF160QG" (at 203.2 80.01 0)
+      (effects (font (size 1.27 1.27)) hide)
+    )
+    (property "Datasheet" "https://www.mouser.mx/datasheet/2/140/TL3305-2065758.pdf" (at 203.2 80.01 0)
+      (effects (font (size 1.27 1.27)) hide)
+    )
+    (property "Manf#" "TL3305AF260QG" (at 203.2 85.09 0)
       (effects (font (size 1.27 1.27)) hide)
     )
@@
       (effects (font (size 1.27 1.27)) hide)
     )
-    (property "LCSC#" "C2886897" (at 203.2 85.09 0)
-      (effects (font (size 1.27 1.27)) hide)
-    )
+    (property "LCSC#" "" (at 203.2 85.09 0)
+      (effects (font (size 1.27 1.27)) hide)
+    )

Commit message: Change manf# of Q4 and Y1
Parts:
- Q4: Manf# RGT16NL65DGTL -> RGT16BM65DTL
- Y1: LCSC# C709001 -> (none); Manf# (none) -> 445I23D12M00000; Proveedor LCSC -> MOUSER
Changed lines of the file:
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@@
       (effects (font (size 1.27 1.27)) (justify left) hide)
     )
-    (property "Datasheet" "https://fscdn.rohm.com/en/products/databook/datasheet/discrete/igbt/rgt16nl65d-e.pdf" (at 150.495 84.455 0)
+    (property "Datasheet" "https://fscdn.rohm.com/en/products/databook/datasheet/discrete/igbt/rgt16bm65d-e.pdf" (at 150.495 84.455 0)
       (effects (font (size 1.27 1.27)) (justify left) hide)
     )
-    (property "Manf#" "RGT16NL65DGTL" (at 139.065 80.645 0)
+    (property "Manf#" "RGT16BM65DTL" (at 139.065 80.645 0)
       (effects (font (size 1.27 1.27)) hide)
     )
@@
       (effects (font (size 1.27 1.27)) hide)
     )
-    (property "Datasheet" "https://datasheet.lcsc.com/lcsc/2008211534_JWT-CM4012M00020T8188026_C709001.pdf" (at 305.054 172.339 0)
-      (effects (font (size 1.27 1.27)) hide)
-    )
-    (property "LCSC#" "C709001" (at 305.054 172.339 0)
-      (effects (font (size 1.27 1.27)) hide)
-    )
-    (property "Proveedor" "LCSC" (at 305.054 172.339 0)
-      (effects (font (size 1.27 1.27)) hide)
-    )
+    (property "Datasheet" "https://www.mouser.mx/datasheet/2/96/008-0360-0-786290.pdf" (at 305.054 172.339 0)
+      (effects (font (size 1.27 1.27)) hide)
+    )
+    (property "LCSC#" "" (at 305.054 172.339 0)
+      (effects (font (size 1.27 1.27)) hide)
+    )
+    (property "Proveedor" "MOUSER" (at 305.054 172.339 0)
+      (effects (font (size 1.27 1.27)) hide)
+    )
+    (property "Manf#" "445I23D12M00000" (at 305.054 172.339 0)
+      (effects (font (size 1.27 1.27)) hide)
+    )

Commit message: Footprint of battery holder modified and J6 changed
Parts:
- J3, J4, J5: now not fitted
- J6: footprint BuggyCat:JST_S2B-PH-K-S(LF)(SN) -> Connector_PinHeader_2.54mm:PinHeader_1x02_P2.54mm_Vertical; LCSC# C173752 -> (none); Proveedor LCSC -> (none); now not fitted
Changed lines of the file:
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@@
   )
   (symbol (lib_id "Connector_Generic:Conn_01x07") (at 196.85 31.115 0) (mirror y) (unit 1)
-    (in_bom yes) (on_board yes) (dnp no) (fields_autoplaced)
+    (in_bom yes) (on_board yes) (dnp yes) (fields_autoplaced)
     (property "Reference" "J3" (at 196.85 16.51 0)
       (effects (font (size 1.27 1.27)))
@@
   )
   (symbol (lib_id "Connector_Generic:Conn_01x02") (at 320.04 38.735 0) (unit 1)
-    (in_bom yes) (on_board yes) (dnp no) (fields_autoplaced)
+    (in_bom yes) (on_board yes) (dnp yes) (fields_autoplaced)
     (property "Reference" "J4" (at 324.485 38.7349 0)
       (effects (font (size 1.27 1.27)) (justify left))
@@
   )
   (symbol (lib_id "Connector_Generic:Conn_01x04") (at 320.04 50.165 0) (unit 1)
-    (in_bom yes) (on_board yes) (dnp no) (fields_autoplaced)
+    (in_bom yes) (on_board yes) (dnp yes) (fields_autoplaced)
     (property "Reference" "J5" (at 324.485 50.1649 0)
       (effects (font (size 1.27 1.27)) (justify left))
@@
   )
   (symbol (lib_id "Connector_Generic:Conn_01x02") (at 368.554 42.672 0) (unit 1)
-    (in_bom yes) (on_board yes) (dnp no) (fields_autoplaced)
+    (in_bom yes) (on_board yes) (dnp yes) (fields_autoplaced)
     (property "Reference" "J6" (at 372.364 42.6719 0)
       (effects (font (size 1.27 1.27)) (justify left))
@@
       (effects (font (size 1.27 1.27)) (justify left))
     )
-    (property "Footprint" "BuggyCat:JST_S2B-PH-K-S(LF)(SN)" (at 368.554 42.672 0)
+    (property "Footprint" "Connector_PinHeader_2.54mm:PinHeader_1x02_P2.54mm_Vertical" (at 368.554 42.672 0)
       (effects (font (size 1.27 1.27)) hide)
     )
@@
       (effects (font (size 1.27 1.27)) hide)
     )
-    (property "LCSC#" "C173752" (at 368.554 42.672 0)
-      (effects (font (size 1.27 1.27)) hide)
-    )
-    (property "Proveedor" "LCSC" (at 368.554 42.672 0)
-      (effects (font (size 1.27 1.27)) hide)
-    )
+    (property "LCSC#" "" (at 368.554 42.672 0)
+      (effects (font (size 1.27 1.27)) hide)
+    )
+    (property "Proveedor" "" (at 368.554 42.672 0)
+      (effects (font (size 1.27 1.27)) hide)
+    )
