File: Hardware/FaultyCat.kicad_sch (KiCad schematic)
At the start: 93 parts, among them J1 Antenna, J10 TRIGGER_VREF, J2 BG306-02-A-2-0400-L-G, J3 Conn_01x10, J4 Header 2, J5 Header 4, J6 Input Power:2x AA Battery, J7 GLITCHER_EN, J8 ANALOG_PINS, J9 TRIGGER_IN, P1 USB_C_Plug_USB2.0, Q1 AO3422, Q1 DMG3415U-7, Q2 AO3422, Q3 LDA111STR, Q4 RGT16BM65DTL, Q7 IRLML2502, Q8 IRF7807PBF, SW1 TL3305AF260QG, SW2 ON, SW3 TL3305AF260QG, SW4 RESET, SW5 BOOT, SW6 TL3305AF260QG, SW7 SW_SP3T, T1 ATB322524, T2 ATB322524, U1 AP2112K-3.3, U2 W25Q16JV, U3 RP2040, U4 TXS0108EPW, U5 TLV75718PDBV, U6 SN74LVC1T45DBV, Y1 12Mhz

Commit message: feat(Hw): update BOM
Parts:
- C1, C10, C13, C2, C3, C5, C6, C8, C9, D7, D8, D9, F1, R1, R13, R14, R16, R2, R3, R4, R5, R6, R7, R8, R9, U3: Proveedor MOUSER -> LCSC
- C11, C12, C14, C15, C16, C17, C18, C19, C20, C7: value 0.1uF -> 100nF; Proveedor MOUSER -> LCSC
- C21, C22: value 0.1uF -> 100nF; LCSC# C26413 -> C66501; Manf# CL10A105KP8NNNC -> (none); Proveedor MOUSER -> LCSC
- J10, J7, J8, J9: Manf# (none) -> 2-PIN
- J3: Manf# (none) -> 10-PIN
- P1: LCSC# C2987386 -> C393939
- Q7, Q8, R23, R24, R25, R26, SW7, U5, U6: Proveedor (none) -> LCSC
- R15: LCSC# (none) -> C116697; Proveedor (none) -> LCSC
- U4: LCSC# C17206 -> C1021790; Proveedor (none) -> LCSC

Commit message: feat: delete dnp resistor
Parts:
- removed R22: R, Resistor_SMD:R_0603_1608Metric, symbol Device:R
- R21: value R -> 10k; LCSC# (none) -> C103199; Proveedor (none) -> LCSC; now fitted
- renumbered D4 to D6, Q1 to Q5, R14 to R12

Commit message: feat(hw): change selector switch
Parts:
- SW7: footprint Button_Switch_SMD:SW_SP3T_PCM13 -> BuggyCat:Sw3P1T; LCSC# C2681567 -> C361168
Changed lines of the file:
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@@
 			)
 		)
-		(property "Footprint" "Button_Switch_SMD:SW_SP3T_PCM13"
+		(property "Footprint" "BuggyCat:Sw3P1T"
 			(at 193.675 208.915 0)
 			(effects
@@
 			)
 		)
-		(property "LCSC#" "C2681567"
+		(property "LCSC#" "C361168"
 			(at 177.8 204.47 0)
 			(effects

Commit message: fix(hw): remove manuf# from P1
Parts:
- P1: Manf# TYPE-C-31-M-31 -> (none)
Changed lines of the file:
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@@
 			)
 		)
-		(property "Manf#" "TYPE-C-31-M-31"
+		(property "Manf#" ""
 			(at 25.4 254.635 0)
 			(effects

Commit message: feat(Hw):Bom_Updated
Parts:
- C11, C12, C14, C15, C16, C17, C18, C19, C20, C7: LCSC# C106209 -> C14663; Manf# CC0402ZRY5V7BB104 -> (none)
- C21, C22: LCSC# C66501 -> C14663
- Q4: LCSC# (none) -> C3193927
Changed lines of the file:
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@@
 			)
 		)
-		(property "LCSC#" "C106209"
+		(property "LCSC#" "C14663"
 			(at 353.695 235.331 0)
 			(effects
@@
 			)
 		)
-		(property "Manf#" "CC0402ZRY5V7BB104"
+		(property "Manf#" ""
 			(at 353.695 235.331 0)
 			(effects
@@
 			)
 		)
-		(property "LCSC#" "C66501"
+		(property "LCSC#" "C14663"
 			(at 241.3 190.5 0)
 			(effects
@@
 			)
 		)
-		(property "LCSC#" "C106209"
+		(property "LCSC#" "C14663"
 			(at 321.437 235.077 0)
 			(effects
@@
 			)
 		)
-		(property "Manf#" "CC0402ZRY5V7BB104"
+		(property "Manf#" ""
 			(at 321.437 235.077 0)
 			(effects
@@
 			)
 		)
+		(property "LCSC#" "C3193927 "
+			(at 139.065 80.645 0)
+			(effects
+				(font
+					(size 1.27 1.27)
+				)
+				(hide yes)
+			)
+		)
 		(pin "1"
 		)
@@
 			)
 		)
-		(property "LCSC#" "C106209"
+		(property "LCSC#" "C14663"
 			(at 391.795 235.331 0)
 			(effects
@@
 			)
 		)
-		(property "Manf#" "CC0402ZRY5V7BB104"
+		(property "Manf#" ""
 			(at 391.795 235.331 0)
 			(effects
@@
 			)
 		)
-		(property "LCSC#" "C106209"
+		(property "LCSC#" "C14663"
 			(at 361.061 235.331 0)
 			(effects
@@
 			)
 		)
-		(property "Manf#" "CC0402ZRY5V7BB104"
+		(property "Manf#" ""
 			(at 361.061 235.331 0)
 			(effects
@@
 			)
 		)
-		(property "LCSC#" "C106209"
+		(property "LCSC#" "C14663"
 			(at 399.415 235.077 0)
 			(effects
@@
 			)
 		)
-		(property "Manf#" "CC0402ZRY5V7BB104"
+		(property "Manf#" ""
 			(at 399.415 235.077 0)
 			(effects
@@
 			)
 		)
-		(property "LCSC#" "C106209"
+		(property "LCSC#" "C14663"
 			(at 368.681 235.331 0)
 			(effects
@@
 			)
 		)
-		(property "Manf#" "CC0402ZRY5V7BB104"
+		(property "Manf#" ""
 			(at 368.681 235.331 0)
 			(effects
@@
 			)
 		)
-		(property "LCSC#" "C106209"
+		(property "LCSC#" "C14663"
 			(at 328.549 235.077 0)
 			(effects
@@
 			)
 		)
-		(property "Manf#" "CC0402ZRY5V7BB104"
+		(property "Manf#" ""
 			(at 328.549 235.077 0)
 			(effects
@@
 			)
 		)
-		(property "LCSC#" "C106209"
+		(property "LCSC#" "C14663"
 			(at 384.175 235.331 0)
 			(effects
@@
 			)
 		)
-		(property "Manf#" "CC0402ZRY5V7BB104"
+		(property "Manf#" ""
 			(at 384.175 235.331 0)
 			(effects
@@
 			)
 		)
-		(property "LCSC#" "C106209"
+		(property "LCSC#" "C14663"
 			(at 376.301 235.331 0)
 			(effects
@@
 			)
 		)
-		(property "Manf#" "CC0402ZRY5V7BB104"
+		(property "Manf#" ""
 			(at 376.301 235.331 0)
 			(effects
@@
 			)
 		)
-		(property "LCSC#" "C106209"
+		(property "LCSC#" "C14663"
 			(at 235.585 273.177 0)
 			(effects
@@
 			)
 		)
-		(property "Manf#" "CC0402ZRY5V7BB104"
+		(property "Manf#" ""
 			(at 235.585 273.177 0)
 			(effects
@@
 			)
 		)
-		(property "LCSC#" "C66501"
+		(property "LCSC#" "C14663"
 			(at 259.08 190.5 0)
 			(effects

Commit message: feat(Hw):Update_BOM
Parts:
- C11, C12, C14, C15, C16, C17, C18, C19, C20, C7: LCSC# C14663 -> C131394
- Q4: LCSC# C3193927 -> (none)
- SW4, SW5: LCSC# C2886897 -> C318889
Changed lines of the file:
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@@
 			)
 		)
-		(property "LCSC#" "C14663"
+		(property "LCSC#" "C131394"
 			(at 353.695 235.331 0)
 			(effects
@@
 			)
 		)
-		(property "LCSC#" "C2886897"
+		(property "LCSC#" "C318889"
 			(at 211.455 276.987 0)
 			(effects
@@
 			)
 		)
-		(property "LCSC#" "C14663"
+		(property "LCSC#" "C131394"
 			(at 321.437 235.077 0)
 			(effects
@@
 			)
 		)
-		(property "LCSC#" "C3193927 "
+		(property "LCSC#" ""
 			(at 139.065 80.645 0)
 			(effects
@@
 			)
 		)
-		(property "LCSC#" "C14663"
+		(property "LCSC#" "C131394"
 			(at 391.795 235.331 0)
 			(effects
@@
 			)
 		)
-		(property "LCSC#" "C14663"
+		(property "LCSC#" "C131394"
 			(at 361.061 235.331 0)
 			(effects
@@
 			)
 		)
-		(property "LCSC#" "C14663"
+		(property "LCSC#" "C131394"
 			(at 399.415 235.077 0)
 			(effects
@@
 			)
 		)
-		(property "LCSC#" "C14663"
+		(property "LCSC#" "C131394"
 			(at 368.681 235.331 0)
 			(effects
@@
 			)
 		)
-		(property "LCSC#" "C14663"
+		(property "LCSC#" "C131394"
 			(at 328.549 235.077 0)
 			(effects
@@
 			)
 		)
-		(property "LCSC#" "C14663"
+		(property "LCSC#" "C131394"
 			(at 384.175 235.331 0)
 			(effects
@@
 			)
 		)
-		(property "LCSC#" "C2886897"
+		(property "LCSC#" "C318889"
 			(at 210.82 264.922 0)
 			(effects
@@
 			)
 		)
-		(property "LCSC#" "C14663"
+		(property "LCSC#" "C131394"
 			(at 376.301 235.331 0)
 			(effects
@@
 			)
 		)
-		(property "LCSC#" "C14663"
+		(property "LCSC#" "C131394"
 			(at 235.585 273.177 0)
 			(effects

Commit message: feat(hw):added_component_replacement
Parts:
- C4: LCSC# (none) -> C692326
- D1, D10, D2, D3: LCSC# (none) -> C437593; Manf# SM4005PL-TP -> 1N4005
- D5: LCSC# (none) -> C263147
- J10, J7, J8, J9: LCSC# (none) -> C7499322
- J3: LCSC# (none) -> C5116489
- Q4: LCSC# (none) -> C3193927
- SW1, SW3, SW6: LCSC# (none) -> C2886902
Changed lines of the file:
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@@
 			)
 		)
-		(property "LCSC#" ""
+		(property "LCSC#" "C2886902"
 			(at 125.73 31.75 0)
 			(effects
@@
 			)
 		)
+		(property "LCSC#" "C5116489"
+			(at 217.17 213.36 0)
+			(effects
+				(font
+					(size 1.27 1.27)
+				)
+				(hide yes)
+			)
+		)
 		(pin "7"
 		)
@@
 			)
 		)
+		(property "LCSC#" "C7499322"
+			(at 36.83 201.93 0)
+			(effects
+				(font
+					(size 1.27 1.27)
+				)
+				(hide yes)
+			)
+		)
 		(pin "2"
 		)
@@
 			)
 		)
+		(property "LCSC#" "C7499322"
+			(at 36.83 196.85 0)
+			(effects
+				(font
+					(size 1.27 1.27)
+				)
+				(hide yes)
+			)
+		)
 		(pin "2"
 		)
@@
 			)
 		)
-		(property "LCSC#" ""
+		(property "LCSC#" "C3193927"
 			(at 139.065 80.645 0)
 			(effects
@@
 			)
 		)
+		(property "LCSC#" "C692326"
+			(at 123.825 74.295 0)
+			(effects
+				(font
+					(size 1.27 1.27)
+				)
+				(hide yes)
+			)
+		)
 		(pin "1"
 		)
@@
 			)
 		)
+		(property "LCSC#" "C7499322"
+			(at 36.83 207.01 0)
+			(effects
+				(font
+					(size 1.27 1.27)
+				)
+				(hide yes)
+			)
+		)
 		(pin "2"
 		)
@@
 			)
 		)
-		(property "Manf#" "SM4005PL-TP"
+		(property "Manf#" "1N4005"
 			(at 368.3 21.59 0)
 			(effects
@@
 			)
 		)
+		(property "LCSC#" "C437593"
+			(at 368.3 21.59 0)
+			(effects
+				(font
+					(size 1.27 1.27)
+				)
+				(hide yes)
+			)
+		)
 		(pin "1"
 		)
@@
 			)
 		)
-		(property "LCSC#" ""
+		(property "LCSC#" "C2886902"
 			(at 331.47 27.305 0)
 			(effects
@@
 			)
 		)
-		(property "Manf#" "SM4005PL-TP"
+		(property "Manf#" "1N4005"
 			(at 46.355 100.965 0)
 			(effects
@@
 			)
 		)
+		(property "LCSC#" "C437593"
+			(at 46.355 100.965 0)
+			(effects
+				(font
+					(size 1.27 1.27)
+				)
+				(hide yes)
+			)
+		)
 		(pin "1"
 		)
@@
 			)
 		)
+		(property "LCSC#" "C7499322"
+			(at 36.83 191.77 0)
+			(effects
+				(font
+					(size 1.27 1.27)
+				)
+				(hide yes)
+			)
+		)
 		(pin "2"
 		)
@@
 			)
 		)
-		(property "Manf#" "SM4005PL-TP"
+		(property "Manf#" "1N4005"
 			(at 23.495 118.745 0)
 			(effects
@@
 			)
 		)
+		(property "LCSC#" "C437593"
+			(at 23.495 118.745 0)
+			(effects
+				(font
+					(size 1.27 1.27)
+				)
+				(hide yes)
+			)
+		)
 		(pin "1"
 		)
@@
 			)
 		)
+		(property "LCSC#" "C263147"
+			(at 126.365 127 90)
+			(effects
+				(font
+					(size 1.27 1.27)
+				)
+				(hide yes)
+			)
+		)
 		(pin "1"
 		)
@@
 			)
 		)
-		(property "LCSC#" ""
+		(property "LCSC#" "C2886902"
 			(at 332.105 83.82 0)
 			(effects
@@
 			)
 		)
-		(property "Manf#" "SM4005PL-TP"
+		(property "Manf#" "1N4005"
 			(at 43.18 147.955 0)
 			(effects
@@
 			(at 43.18 147.955 0)
 			(effects
+				(font
+					(size 1.27 1.27)
+				)
+				(hide yes)
+			)
+		)
+		(property "LCSC#" "C437593"
+			(at 43.18 147.955 0)
+			(effects
